Commit message: Main

File: src/abb_experimental/abb_irb140_gazebo/urdf/irb140_macro.xacro (robot description, xacro)
@@ -5,60 +5,4 @@
   <!-- get base ABB IRB120 model -->
   <xacro:abb_irb140 prefix="${prefix}" />
-  <!-- transmission list -->
-  <transmission name="${prefix}tran1">
-    <type>transmission_interface/SimpleTransmission</type>
-    <joint name="${prefix}joint_1">
-      <hardwareInterface>hardware_interface/PositionJointInterface</hardwareInterface>
-    </joint>
-    <actuator name="${prefix}motor1">
-      <mechanicalReduction>1</mechanicalReduction>
-    </actuator>
-  </transmission>
-  <transmission name="${prefix}tran2">
-    <type>transmission_interface/SimpleTransmission</type>
-    <joint name="${prefix}joint_2">
-      <hardwareInterface>PositionJointInterface</hardwareInterface>
-    </joint>
-    <actuator name="${prefix}motor2">
-      <mechanicalReduction>1</mechanicalReduction>
-    </actuator>
-  </transmission>
-  <transmission name="${prefix}tran3">
-    <type>transmission_interface/SimpleTransmission</type>
-    <joint name="${prefix}joint_3">
-      <hardwareInterface>PositionJointInterface</hardwareInterface>
-    </joint>
-    <actuator name="${prefix}motor3">
-      <mechanicalReduction>1</mechanicalReduction>
-    </actuator>
-  </transmission>
-  <transmission name="${prefix}tran4">
-    <type>transmission_interface/SimpleTransmission</type>
-    <joint name="${prefix}joint_4">
-      <hardwareInterface>PositionJointInterface</hardwareInterface>
-    </joint>
-    <actuator name="${prefix}motor4">
-      <mechanicalReduction>1</mechanicalReduction>
-    </actuator>
-  </transmission>
-  <transmission name="${prefix}tran5">
-    <type>transmission_interface/SimpleTransmission</type>
-    <joint name="${prefix}joint_5">
-      <hardwareInterface>PositionJointInterface</hardwareInterface>
-    </joint>
-    <actuator name="${prefix}motor5">
-      <mechanicalReduction>1</mechanicalReduction>
-    </actuator>
-  </transmission>
-  <transmission name="${prefix}tran6">
-    <type>transmission_interface/SimpleTransmission</type>
-    <joint name="${prefix}joint_6">
-      <hardwareInterface>PositionJointInterface</hardwareInterface>
-    </joint>
-    <actuator name="${prefix}motor6">
-      <mechanicalReduction>1</mechanicalReduction>
-    </actuator>
-  </transmission>
-  <!-- end of transmission list -->
   <!-- Gazebo-specific link properties -->
   <gazebo reference="${prefix}base_link">
@@ -90,4 +34,60 @@
     <turnGravityOff>true</turnGravityOff>
   </gazebo>
+  <!-- transmission list -->
+  <transmission name="${prefix}tran1">
+    <type>transmission_interface/SimpleTransmission</type>
+    <joint name="${prefix}joint_1">
+      <hardwareInterface>hardware_interface/PositionJointInterface</hardwareInterface>
+    </joint>
+    <actuator name="${prefix}motor1">
+      <mechanicalReduction>1</mechanicalReduction>
+    </actuator>
+  </transmission>
+  <transmission name="${prefix}tran2">
+    <type>transmission_interface/SimpleTransmission</type>
+    <joint name="${prefix}joint_2">
+      <hardwareInterface>hardware_interface/PositionJointInterface</hardwareInterface>
+    </joint>
+    <actuator name="${prefix}motor2">
+      <mechanicalReduction>1</mechanicalReduction>
+    </actuator>
+  </transmission>
+  <transmission name="${prefix}tran3">
+    <type>transmission_interface/SimpleTransmission</type>
+    <joint name="${prefix}joint_3">
+      <hardwareInterface>hardware_interface/PositionJointInterface</hardwareInterface>
+    </joint>
+    <actuator name="${prefix}motor3">
+      <mechanicalReduction>1</mechanicalReduction>
+    </actuator>
+  </transmission>
+  <transmission name="${prefix}tran4">
+    <type>transmission_interface/SimpleTransmission</type>
+    <joint name="${prefix}joint_4">
+      <hardwareInterface>hardware_interface/PositionJointInterface</hardwareInterface>
+    </joint>
+    <actuator name="${prefix}motor4">
+      <mechanicalReduction>1</mechanicalReduction>
+    </actuator>
+  </transmission>
+  <transmission name="${prefix}tran5">
+    <type>transmission_interface/SimpleTransmission</type>
+    <joint name="${prefix}joint_5">
+      <hardwareInterface>hardware_interface/PositionJointInterface</hardwareInterface>
+    </joint>
+    <actuator name="${prefix}motor5">
+      <mechanicalReduction>1</mechanicalReduction>
+    </actuator>
+  </transmission>
+  <transmission name="${prefix}tran6">
+    <type>transmission_interface/SimpleTransmission</type>
+    <joint name="${prefix}joint_6">
+      <hardwareInterface>hardware_interface/PositionJointInterface</hardwareInterface>
+    </joint>
+    <actuator name="${prefix}motor6">
+      <mechanicalReduction>1</mechanicalReduction>
+    </actuator>
+  </transmission>
+  <!-- end of transmission list -->
   <!-- ros_control plugin -->
   <gazebo>

File: src/abb_experimental/abb_irb140_support/urdf/irb140_macro.xacro (robot description, xacro)
@@ -2,5 +2,5 @@
 <robot xmlns:xacro="http://ros.org/wiki/xacro">
 <xacro:macro name="abb_irb140" params="prefix">
-    <!-- link list -->
+<!--Se comenzara en orden desde el base_link hasta la herramienta-->
     <link name="${prefix}base_link">
         <visual>
@@ -21,104 +21,10 @@
             </material>
         </collision>
-    </link>
-    <link name="${prefix}link_1">
-        <visual>
-            <origin xyz="0 0 0" rpy="0 0 0"/>
-            <geometry>
-                <mesh filename="package://abb_irb140_support/meshes/irb140/visual/link_1.stl"/>
-            </geometry>
-            <material name="abb_orange"/>
-        </visual>
-        <collision>
-            <origin xyz="0 0 0" rpy="0 0 0"/>
-            <geometry>
-                <mesh filename="package://abb_irb140_support/meshes/irb140/collision/link_1.stl"/>
-            </geometry>
-            <material name="yellow"/>
-        </collision>
-    </link>
-    <link name="${prefix}link_2">
-        <visual>
-            <origin xyz="0 0 0" rpy="0 0 0"/>
-            <geometry>
-                <mesh filename="package://abb_irb140_support/meshes/irb140/visual/link_2.stl"/>
-            </geometry>
-            <material name="abb_orange"/>
-        </visual>
-        <collision>
-            <origin xyz="0 0 0" rpy="0 0 0"/>
-            <geometry>
-                <mesh filename="package://abb_irb140_support/meshes/irb140/collision/link_2.stl"/>
-            </geometry>
-            <material name="yellow"/>
-        </collision>
-    </link>
-    <link name="${prefix}link_3">
-        <visual>
-            <origin xyz="0 0 0" rpy="0 0 0"/>
-            <geometry>
-                <mesh filename="package://abb_irb140_support/meshes/irb140/visual/link_3.stl"/>
-            </geometry>
-            <material name="abb_orange"/>
-        </visual>
-        <collision>
-            <origin xyz="0 0 0" rpy="0 0 0"/>
-            <geometry>
-                <mesh filename="package://abb_irb140_support/meshes/irb140/collision/link_3.stl"/>
-            </geometry>
-            <material name="yellow"/>
-        </collision>
-    </link>
-    <link name="${prefix}link_4">
-        <visual>
-            <origin xyz="0 0 0" rpy="0 0 0"/>
-            <geometry>
-                <mesh filename="package://abb_irb140_support/meshes/irb140/visual/link_4.stl"/>
-            </geometry>
-            <material name="abb_orange"/>
-        </visual>
-        <collision>
-            <origin xyz="0 0 0" rpy="0 0 0"/>
-            <geometry>
-                <mesh filename="package://abb_irb140_support/meshes/irb140/collision/link_4.stl"/>
-            </geometry>
-            <material name="yellow"/>
-        </collision>
-    </link>
-    <link name="${prefix}link_5">
-        <visual>
-            <origin xyz="0 0 0" rpy="0 0 0"/>
-            <geometry>
-                <mesh filename="package://abb_irb140_support/meshes/irb140/visual/link_5.stl"/>
-            </geometry>
-            <material name="abb_orange"/>
-        </visual>
-        <collision>
-            <origin xyz="0 0 0" rpy="0 0 0"/>
-            <geometry>
-                <mesh filename="package://abb_irb140_support/meshes/irb140/collision/link_5.stl"/>
-            </geometry>
-            <material name="yellow"/>
-        </collision>
-    </link>
-    <link name="${prefix}link_6">
-        <visual>
-            <origin xyz="0 0 0" rpy="0 0 0"/>
-            <geometry>
-                <mesh filename="package://abb_irb140_support/meshes/irb140/visual/link_6.stl"/>
-            </geometry>
-            <material name="abb_orange"/>
-        </visual>
-        <collision>
-            <origin xyz="0 0 0" rpy="0 0 0"/>
-            <geometry>
-                <mesh filename="package://abb_irb140_support/meshes/irb140/collision/link_6.stl"/>
-            </geometry>
-            <material name="yellow"/>
-        </collision>
-    </link>
-    <link name="${prefix}tool0"/>
-    <!-- end of link list -->
-    <!-- joint list -->
+        <inertial>
+            <mass value="6.215"/>
+            <origin xyz="-0.04204 8.01E-05 0.07964" rpy="0 0 0"/>
+            <inertia ixx="0.0247272" ixy="-8.0784E-05" ixz="0.00130902" iyy="0.0491285" iyz="-8.0419E-06" izz="0.0472376"/>
+        </inertial>
+    </link>
     <joint name="${prefix}joint_1" type="revolute">
         <origin xyz="0 0 0" rpy="0 0 0"/>
@@ -128,6 +34,28 @@
         <limit lower="-3.1416" upper="3.1416" effort="0" velocity="2.618"/>
     </joint>
+    <link name="${prefix}link_1">
+        <visual>
+            <origin xyz="0 0 0" rpy="0 0 0"/>
+            <geometry>
+                <mesh filename="package://abb_irb140_support/meshes/irb140/visual/link_1.stl"/>
+            </geometry>
+            <material name="abb_orange"/>
+        </visual>
+        <collision>
+            <origin xyz="0 0 0" rpy="0 0 0"/>
+            <geometry>
+                <mesh filename="package://abb_irb140_support/meshes/irb140/collision/link_1.stl"/>
+            </geometry>
+            <material name="yellow"/>
+        </collision>
+    <inertial>
+        <mass value="3.067" />
+        <origin xyz="0 0 0" rpy="0 0 0"/>
+        <!--origin xyz="9.77E-05 -0.00012 0.23841" rpy="0 0 0"/-->
+        <inertia ixx="0.0142175" ixy="-1.28579E-05" ixz="-2.31364E-05" iyy="0.0144041" iyz="1.93404E-05" izz="0.0104533"/>
+    </inertial>
+    </link>
     <joint name="${prefix}joint_2" type="revolute">
-        <origin xyz="0.1 0 0.615" rpy="0 0 0"/>
+        <origin xyz="0.28 0 1.38" rpy="0 0 0"/>
         <parent link="${prefix}link_1"/>
         <child link="${prefix}link_2"/>
@@ -135,6 +63,28 @@
         <limit lower="-1.7453" upper="1.9199" effort="0" velocity="2.618"/>
     </joint>
+    <link name="${prefix}link_2">
+        <visual>
+            <origin xyz="-0.28 0 -1.38" rpy="0 0 0"/>
+            <geometry>
+                <mesh filename="package://abb_irb140_support/meshes/irb140/visual/link_2.stl"/>
+            </geometry>
+            <material name="abb_orange"/>
+        </visual>
+        <collision>
+            <origin xyz="-0.28 0 -1.38" rpy="0 0 0"/>
+            <geometry>
+                <mesh filename="package://abb_irb140_support/meshes/irb140/collision/link_2.stl"/>
+            </geometry>
+            <material name="yellow"/>
+        </collision>
+        <inertial>
+            <mass value="3.909"/>
+            <origin xyz="0 0 0" rpy="0 0 0"/>
+            <!--origin xyz="0.00078 -0.00212 0.10124" rpy="0 0 0"/-->
+            <inertia ixx="0.0603111" ixy="9.83431E-06" ixz="5.72407E-05" iyy="0.041569" iyz="-0.00050497" izz="0.0259548"/>
+        </inertial>
+    </link>
     <joint name="${prefix}joint_3" type="revolute">
-        <origin xyz="0 0 0.705" rpy="0 0 0"/>
+        <origin xyz="0 0 1.42" rpy="0 0 0"/>
         <parent link="${prefix}link_2"/>
         <child link="${prefix}link_3"/>
@@ -142,6 +92,28 @@
         <limit lower="-1.0472" upper="1.1345" effort="0" velocity="2.618"/>
     </joint>
-    <joint name="${prefix}joint_4" type="revolute">
-        <origin xyz="0.258 0 0.135" rpy="0 0 0"/>
+    <link name="${prefix}link_3">
+        <visual>
+            <origin xyz="-0.28 0 -2.8" rpy="0 0 0"/>
+            <geometry>
+                <mesh filename="package://abb_irb140_support/meshes/irb140/visual/link_3.stl"/>
+            </geometry>
+            <material name="abb_orange"/>
+        </visual>
+        <collision>
+            <origin xyz="-0.28 0 -2.8" rpy="0 0 0"/>
+            <geometry>
+                <mesh filename="package://abb_irb140_support/meshes/irb140/collision/link_3.stl"/>
+            </geometry>
+            <material name="yellow"/>
+        </collision>
+      <inertial>
+         <mass value="2.944"/>
+         <origin xyz="0 0 0" rpy="0 0 0"/>
+         <!--origin xyz="0.02281 0.00106 0.05791" rpy="0 0 0"/-->
+         <inertia ixx="0.00835606" ixy="-8.01545E-05" ixz="0.00142884" iyy="0.016713" iyz="-0.000182227" izz="0.0126984"/>
+      </inertial>
+    </link>
+ <joint name="${prefix}joint_4" type="revolute">
+        <origin xyz="0 0 0" rpy="0 0 0"/>
         <parent link="${prefix}link_3"/>
         <child link="${prefix}link_4"/>
@@ -149,6 +121,28 @@
         <limit lower="-3.49" upper="3.49" effort="0" velocity="6.2832"/>
     </joint>
-    <joint name="${prefix}joint_5" type="revolute">
-        <origin xyz="0.497 0 0" rpy="0 0 0"/>
+    <link name="${prefix}link_4">
+        <visual>
+            <origin xyz="-0.28 0 -2.8" rpy="0 0 0"/>
+            <geometry>
+                <mesh filename="package://abb_irb140_support/meshes/irb140/visual/link_4.stl"/>
+            </geometry>
+            <material name="abb_orange"/>
+        </visual>
+        <collision>
+            <origin xyz="-0.28 0 -2.8" rpy="0 0 0"/>
+            <geometry>
+                <mesh filename="package://abb_irb140_support/meshes/irb140/collision/link_4.stl"/>
+            </geometry>
+            <material name="yellow"/>
+        </collision>
+       <inertial>
+        <mass value="1.328"/>
+        <origin xyz="0.2247 0.00015 0.00041" rpy="0 0 0"/>
+        <!--origin xyz="0.2247 0.00015 0.00041" rpy="0 0 0"/-->
+        <inertia ixx="0.00284661" ixy="-2.12765E-05" ixz="-1.6435E-05" iyy="0.00401346" iyz="1.31336E-05" izz="0.0052535"/>
+      </inertial>
+    </link>
+ <joint name="${prefix}joint_5" type="revolute">
+        <origin xyz="1.49 0 0" rpy="0 0 0"/>
         <parent link="${prefix}link_4"/>
         <child link="${prefix}link_5"/>
@@ -156,6 +150,27 @@
         <limit lower="-2.0944" upper="2.0944" effort="0" velocity="6.2832"/>
     </joint>
-    <joint name="${prefix}joint_6" type="revolute">
-        <origin xyz="0.085 0 0" rpy="0 0 0"/>
+    <link name="${prefix}link_5">
+        <visual>
+            <origin xyz="-1.77 0 -2.8" rpy="0 0 0"/>
+            <geometry>
+                <mesh filename="package://abb_irb140_support/meshes/irb140/visual/link_5.stl"/>
+            </geometry>
+            <material name="abb_orange"/>
+        </visual>
+        <collision>
+            <origin xyz="-1.77 0 -2.8" rpy="0 0 0"/>
+            <geometry>
+                <mesh filename="package://abb_irb140_support/meshes/irb140/collision/link_5.stl"/>
+            </geometry>
+            <material name="yellow"/>
+        </collision>
+       <inertial>
+        <mass value="0.546"/>
+        <origin xyz="-0.00109 3.68E-05 6.22E-05" rpy="0 0 0"/>
+        <inertia ixx="0.000404891" ixy="1.61943E-06" ixz="8.46805E-07" iyy="0.000892825" iyz="-1.51792E-08" izz="0.000815468"/>
+       </inertial>
+    </link>
+  <joint name="${prefix}joint_6" type="revolute">
+        <origin xyz="0 0 0.02" rpy="0 0 0"/>
         <parent link="${prefix}link_5"/>
         <child link="${prefix}link_6"/>
@@ -163,4 +178,25 @@
         <limit lower="-6.9813" upper="6.9813" effort="0" velocity="7.854"/>
     </joint>
+    <link name="${prefix}link_6">
+        <visual>
+            <origin xyz="-1.77 0 -2.8" rpy="0 0 0"/>
+            <geometry>
+                <mesh filename="package://abb_irb140_support/meshes/irb140/visual/link_6.stl"/>
+            </geometry>
+            <material name="abb_orange"/>
+        </visual>
+        <collision>
+            <origin xyz="-1.77 0 -2.8" rpy="0 0 0"/>
+            <geometry>
+                <mesh filename="package://abb_irb140_support/meshes/irb140/collision/link_6.stl"/>
+            </geometry>
+            <material name="yellow"/>
+        </collision>
+     <inertial>
+        <mass value="0.137"/>
+        <origin xyz="-0.00706 -0.00017 -1.32E-06" rpy="0 0 0"/>
+        <inertia ixx="0.001" ixy="0" ixz="0" iyy="0.001" iyz="0" izz="0.001"/>
+      </inertial>
+    </link>
     <joint name="${prefix}joint_6-tool0" type="fixed">
         <parent link="${prefix}link_6"/>
@@ -168,4 +204,6 @@
         <origin xyz="0 0 0" rpy="0 1.57079632679 0"/>
     </joint>
+    <link name="${prefix}tool0"/>
+    <!-- end of link list -->
     <!-- end of joint list -->
     <!-- ROS base_link to ABB World Coordinates transform -->
